File: hardware/rx/rx.kicad_sch (KiCad schematic)
At the start: 16 parts, among them J1 Conn_01x04, J3 PPM, J4 AUX2, J6 VIN, SW1 SW_Push, U1 E28-2G4M12S, U3 ESP32-C3_SUPERMINI, U5 MIC5219-3.3YM5

Commit message: rx PCB
Parts:
- added J2: VBAT, unfancyRemote_components:SolderWirePad_1x01_SMD_1x2mm, symbol Connector_Generic:Conn_01x01
- added JP1, JP2, JP3, JP4, JP5, JP6: SolderJumper_2_Open, Jumper:SolderJumper-2_P1.3mm_Open_RoundedPad1.0x1.5mm, symbol Jumper:SolderJumper_2_Open
- added R10, R8: 150K, Resistor_SMD:R_0402_1005Metric, symbol Device:R
- added R11, R7: 3.3K, Resistor_SMD:R_0402_1005Metric, symbol Device:R
- added R2, R6: 120K, Resistor_SMD:R_0402_1005Metric, symbol Device:R
- added R3: 6.8K, Resistor_SMD:R_0402_1005Metric, symbol Device:R
- added R4: 100K, Resistor_SMD:R_0402_1005Metric, symbol Device:R
- added R5, R9: 4.7K, Resistor_SMD:R_0402_1005Metric, symbol Device:R
- R13: value 6.8K -> 5.6K
Connections:
- net GND: now also R11.2, R3.2, R5.2, R7.2, R9.2
- net VBAT: now also J2.1 (Pin_1), JP1.2 (B), JP2.2 (B), JP3.2 (B), JP4.2 (B), JP5.2 (B), JP6.2 (B); no longer R12.1
- net VBATSCALED: now also R10.2, R11.1, R2.2, R3.1, R4.2, R5.1, R6.2, R7.1, R8.2, R9.1
- new net 12S: JP1.1 (A), R12.1
- new net 14S: JP3.1 (A), R4.1
- new net 16S: JP2.1 (A), R2.1
- new net 18S: JP4.1 (A), R6.1
- new net 20S: JP5.1 (A), R8.1
- new net 22S: JP6.1 (A), R10.1
Other:
- moved on the sheet: R12, R13

Commit message: update to kicad 9
Parts:
- removed J6: VIN, unfancyRemote_components:SolderWirePad_1x02_SMD_1x2mm, symbol Connector_Generic:Conn_01x02
Changed lines of the file:
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@@
 (kicad_sch
-	(version 20231120)
+	(version 20250114)
 	(generator "eeschema")
-	(generator_version "8.0")
+	(generator_version "9.0")
 	(paper "A4")
 	(junction
@@
 	(wire
 		(pts
-			(xy 68.58 118.11) (xy 71.12 118.11)
-		)
-		(stroke
-			(width 0)
-			(type default)
-		)
-	)
-	(wire
-		(pts
 			(xy 111.76 85.09) (xy 111.76 46.99)
 		)
@@
 	(wire
 		(pts
-			(xy 66.04 115.57) (xy 71.12 115.57)
-		)
-		(stroke
-			(width 0)
-			(type default)
-		)
-	)
-	(wire
-		(pts
 			(xy 114.3 82.55) (xy 114.3 44.45)
 		)
@@
 	(label "RFBUSY"
 		(at 151.13 87.63 0)
-		(fields_autoplaced yes)
 		(effects
 			(font
@@
 	(label "MISO"
 		(at 116.84 82.55 0)
-		(fields_autoplaced yes)
 		(effects
 			(font
@@
 	(label "MOSI"
 		(at 118.11 85.09 0)
-		(fields_autoplaced yes)
 		(effects
 			(font
@@
 	(label "SCK"
 		(at 120.65 87.63 0)
-		(fields_autoplaced yes)
 		(effects
 			(font
@@
 	(label "NSS"
 		(at 120.65 90.17 0)
-		(fields_autoplaced yes)
 		(effects
 			(font
@@
 	(label "NRESET"
 		(at 151.13 90.17 0)
-		(fields_autoplaced yes)
 		(effects
 			(font
@@
 		)
 	)
-	(global_label "+5V"
-		(shape input)
-		(at 66.04 115.57 180)
-		(fields_autoplaced yes)
-		(effects
-			(font
-				(size 1.27 1.27)
-			)
-			(justify right)
-		)
-		(property "Intersheetrefs" "${INTERSHEET_REFS}"
-			(at 59.1843 115.57 0)
-			(effects
-				(font
-					(size 1.27 1.27)
-				)
-				(justify right)
-				(hide yes)
-			)
-		)
-	)
 	(global_label "PPM"
 		(shape input)
@@
 	)
 	(symbol
-		(lib_id "Connector_Generic:Conn_01x02")
-		(at 76.2 115.57 0)
-		(unit 1)
-		(exclude_from_sim no)
-		(in_bom yes)
-		(on_board yes)
-		(dnp no)
-		(fields_autoplaced yes)
-		(property "Reference" "J6"
-			(at 78.74 115.5699 0)
-			(effects
-				(font
-					(size 1.27 1.27)
-				)
-				(justify left)
-			)
-		)
-		(property "Value" "VIN"
-			(at 78.74 118.1099 0)
-			(effects
-				(font
-					(size 1.27 1.27)
-				)
-				(justify left)
-			)
-		)
-		(property "Footprint" "unfancyRemote_components:SolderWirePad_1x02_SMD_1x2mm"
-			(at 76.2 115.57 0)
-			(effects
-				(font
-					(size 1.27 1.27)
-				)
-				(hide yes)
-			)
-		)
-		(property "Datasheet" "~"
-			(at 76.2 115.57 0)
-			(effects
-				(font
-					(size 1.27 1.27)
-				)
-				(hide yes)
-			)
-		)
-		(property "Description" ""
-			(at 76.2 115.57 0)
-			(effects
-				(font
-					(size 1.27 1.27)
-				)
-				(hide yes)
-			)
-		)
-		(pin "1"
-		)
-		(pin "2"
-		)
-		(instances
-			(project ""
-				(path "/9538e4ed-27e6-4c37-b989-9859dc0d49e8"
-					(reference "J6")
-					(unit 1)
-				)
-			)
-		)
-	)
-	(symbol
 		(lib_id "Device:R")
 		(at 119.38 166.37 0)
@@
 	)
 	(symbol
+		(lib_name "SolderJumper_2_Open_1")
 		(lib_id "Jumper:SolderJumper_2_Open")
 		(at 201.93 109.22 0)
@@
 	)
 	(symbol
-		(lib_id "power:GND")
-		(at 68.58 118.11 270)
-		(unit 1)
-		(exclude_from_sim no)
-		(in_bom yes)
-		(on_board yes)
-		(dnp no)
-		(fields_autoplaced yes)
-		(property "Reference" "#PWR0120"
-			(at 62.23 118.11 0)
-			(effects
-				(font
-					(size 1.27 1.27)
-				)
-				(hide yes)
-			)
-		)
-		(property "Value" "GND"
-			(at 67.31 121.92 90)
-			(effects
-				(font
-					(size 1.27 1.27)
-				)
-			)
-		)
-		(property "Footprint" ""
-			(at 68.58 118.11 0)
-			(effects
-				(font
-					(size 1.27 1.27)
-				)
-				(hide yes)
-			)
-		)
-		(property "Datasheet" ""
-			(at 68.58 118.11 0)
-			(effects
-				(font
-					(size 1.27 1.27)
-				)
-				(hide yes)
-			)
-		)
-		(property "Description" ""
-			(at 68.58 118.11 0)
-			(effects
-				(font
-					(size 1.27 1.27)
-				)
-				(hide yes)
-			)
-		)
-		(pin "1"
-		)
-		(instances
-			(project ""
-				(path "/9538e4ed-27e6-4c37-b989-9859dc0d49e8"
-					(reference "#PWR0120")
-					(unit 1)
-				)
-			)
-		)
-	)
-	(symbol
 		(lib_id "Connector_Generic:Conn_01x03")
 		(at 90.17 72.39 0)
@@
 		)
 	)
+	(embedded_fonts no)
 )
