File: hardware/tx/unfancyRemote.kicad_sch (KiCad schematic)
At the start: 57 parts, among them J1 Battery, J3 HALL1/PPM, J4 HALL2, J6 VIN, J8 Motor, Q1 AO3401A, Q2 MMBT3904, Q3 MMBT3904, SW1 SW_Push, U1 E28-2G4M12S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

Commit message: update to kicad 9
Parts:
- R13: value 6.8K -> 100K
Changed lines of the file:
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@@
 (kicad_sch
-	(version 20231120)
+	(version 20250114)
 	(generator "eeschema")
-	(generator_version "8.0")
+	(generator_version "9.0")
 	(paper "A4")
 	(junction
@@
 	(label "RFBUSY"
 		(at 151.13 87.63 0)
-		(fields_autoplaced yes)
 		(effects
 			(font
@@
 	(label "MISO"
 		(at 116.84 82.55 0)
-		(fields_autoplaced yes)
 		(effects
 			(font
@@
 	(label "MOSI"
 		(at 118.11 85.09 0)
-		(fields_autoplaced yes)
 		(effects
 			(font
@@
 	(label "SCK"
 		(at 120.65 87.63 0)
-		(fields_autoplaced yes)
 		(effects
 			(font
@@
 	(label "NSS"
 		(at 120.65 90.17 0)
-		(fields_autoplaced yes)
 		(effects
 			(font
@@
 	(label "NRESET"
 		(at 151.13 90.17 0)
-		(fields_autoplaced yes)
 		(effects
 			(font
@@
 			)
 		)
-		(property "Value" "6.8K"
+		(property "Value" "100K"
 			(at 90.17 109.2199 0)
 			(effects
@@
 		)
 	)
+	(embedded_fonts no)
 )
